File: mbus_guru.sch (KiCad schematic (older format))
At the start: 40 parts, among them J1 Conn_01x02, J2 Conn_01x02, J3 Conn_01x02, J4 Conn_01x03, Q1 BCV71, Q2 MMBT2907A, Q3 BCV71, Q4 MMBT2907A, Q5 BCV71, U1 74HC14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

Commit message: Fixed bug with transistor footprints
Parts:
- Q1, Q2, Q3, Q4, Q5: footprint Package_TO_SOT_SMD:SOT-23 -> SOT-23-Custom:BCV71_SOT-23_Handsoldering
- TP1: footprint TestPoint:TestPoint_Keystone_5015_Micro-Minature -> TestPoint:TestPoint_Pad_2.0x2.0mm
Connections:
- net Q1E: now reaches C1.1, FB1.2, Q1.3 (E), Q2.3 (E), R9.1
- net Q1C: now reaches C3.1, Q1.1 (C), R2.2, TP1.1
- net Q1B: now reaches C2.1, Q1.2 (B), R1.2, R6.1
Changed lines of the file:
@@
 EESchema Schematic File Version 4
-LIBS:mbus_guru-cache
-EELAYER 29 0
+EELAYER 30 0
 EELAYER END
 $Descr A4 11693 8268
@@
 F 0 "Q3" H 6490 2746 50  0000 L CNN
 F 1 "BCV71" H 6490 2655 50  0000 L CNN
-F 2 "Package_TO_SOT_SMD:SOT-23" H 6500 2625 50  0001 L CIN
+F 2 "SOT-23-Custom:BCV71_SOT-23_Handsoldering" H 6500 2625 50  0001 L CIN
 F 3 "https://diotec.com/tl_files/diotec/files/pdf/datasheets/bc337.pdf" H 6300 2700 50  0001 L CNN
 F 4 "On Semi" H 6300 2700 50  0001 C CNN "MFG Name"
@@
 F 0 "Q2" H 7165 2346 50  0000 L CNN
 F 1 "MMBT2907A" H 7165 2255 50  0000 L CNN
-F 2 "Package_TO_SOT_SMD:SOT-23" H 7175 2225 50  0001 L CIN
+F 2 "SOT-23-Custom:BCV71_SOT-23_Handsoldering" H 7175 2225 50  0001 L CIN
 F 3 "http://www.onsemi.com/pub_link/Collateral/BC327-D.PDF" H 6975 2300 50  0001 L CNN
 F 4 "Diodes Inc" H 6975 2300 50  0001 C CNN "MFG Name"
@@
 F 0 "Q4" H 4990 1996 50  0000 L CNN
 F 1 "MMBT2907A" H 4990 1905 50  0000 L CNN
-F 2 "Package_TO_SOT_SMD:SOT-23" H 5000 1875 50  0001 L CIN
+F 2 "SOT-23-Custom:BCV71_SOT-23_Handsoldering" H 5000 1875 50  0001 L CIN
 F 3 "http://www.onsemi.com/pub_link/Collateral/BC327-D.PDF" H 4800 1950 50  0001 L CNN
 	1    4800 1950
@@
 F 0 "Q1" H 7165 1871 50  0000 L CNN
 F 1 "BCV71" H 7165 1780 50  0000 L CNN
-F 2 "Package_TO_SOT_SMD:SOT-23" H 7175 1750 50  0001 L CIN
+F 2 "SOT-23-Custom:BCV71_SOT-23_Handsoldering" H 7175 1750 50  0001 L CIN
 F 3 "https://diotec.com/tl_files/diotec/files/pdf/datasheets/bc337.pdf" H 6975 1825 50  0001 L CNN
 F 4 "On Semi" H 6975 1825 50  0001 C CNN "MFG Name"
@@
 F 0 "Q5" H 4690 2396 50  0000 L CNN
 F 1 "BCV71" H 4690 2305 50  0000 L CNN
-F 2 "Package_TO_SOT_SMD:SOT-23" H 4700 2275 50  0001 L CIN
+F 2 "SOT-23-Custom:BCV71_SOT-23_Handsoldering" H 4700 2275 50  0001 L CIN
 F 3 "https://diotec.com/tl_files/diotec/files/pdf/datasheets/bc337.pdf" H 4500 2350 50  0001 L CNN
 F 4 "On Semi" H 4500 2350 50  0001 C CNN "MFG Name"
@@
 F 0 "TP1" V 6150 1925 50  0000 C CNN
 F 1 "TestPoint" V 6075 1975 50  0000 C CNN
-F 2 "TestPoint:TestPoint_Keystone_5015_Micro-Minature" H 6350 1675 50  0001 C CNN
+F 2 "TestPoint:TestPoint_Pad_2.0x2.0mm" H 6350 1675 50  0001 C CNN
 F 3 "~" H 6350 1675 50  0001 C CNN
 F 4 "Keystone" H 6150 1675 50  0001 C CNN "MFG Name"
@@
 Text Notes 6025 4550 0    50   ~ 0
 M-Bus short detection. Comparator outputs 3V3 if input is < -33 V.  D3 lights up.
+Text Label 7075 1625 0    50   ~ 0
+Q1C
+Text Label 6400 1825 0    50   ~ 0
+Q1B
+Text Label 7075 2100 0    50   ~ 0
+Q1E
 $EndSCHEMATC

Commit message: Added missing component U1G of 74HC14
Parts:
- added unit 7 of U1
Connections:
- net 3V3: now also U1.14 (VCC)
- net GND: now also U1.7 (GND)
- net Q2B: now reaches Q2.2 (B), R6.2, R8.1
- net Q3C: now reaches Q3.1 (C), R8.2
- net Q3B: now reaches Q3.2 (B), R11.1
- net Q5C: now reaches Q5.1 (C), R4.2, U1.9
- net Q2C: now reaches Q2.1 (C), R10.1
- net Q4B: now reaches C4.1, Q4.2 (B), R3.1
- net Q4C: now reaches Q4.1 (C), R5.1
- net Q5B: now reaches Q5.2 (B), R5.2, R7.1
Other:
- moved on the sheet: R11
Changed lines of the file:
@@
 L Device:R_Small R11
 U 1 1 5E11360F
-P 6000 2700
-F 0 "R11" H 6059 2746 50  0000 L CNN
-F 1 "10k 1%" H 6059 2655 50  0000 L CNN
-F 2 "Resistor_SMD:R_0603_1608Metric" H 6000 2700 50  0001 C CNN
-F 3 "~" H 6000 2700 50  0001 C CNN
-	1    6000 2700
+P 5875 2700
+F 0 "R11" H 5934 2746 50  0000 L CNN
+F 1 "10k 1%" H 5934 2655 50  0000 L CNN
+F 2 "Resistor_SMD:R_0603_1608Metric" H 5875 2700 50  0001 C CNN
+F 3 "~" H 5875 2700 50  0001 C CNN
+	1    5875 2700
 	0    1    1    0
 $EndComp
@@
 Wire Wire Line
 	5525 3225 5525 2700
-Wire Wire Line
-	5525 2700 5900 2700
 Text Label 4275 3225 2    50   ~ 0
 MBUS-TX
@@
 L power:GND #PWR0104
 U 1 1 5E2C9A38
-P 4300 1600
-F 0 "#PWR0104" H 4300 1350 50  0001 C CNN
-F 1 "GND" V 4305 1472 50  0000 R CNN
-F 2 "" H 4300 1600 50  0001 C CNN
-F 3 "" H 4300 1600 50  0001 C CNN
-	1    4300 1600
+P 4225 1600
+F 0 "#PWR0104" H 4225 1350 50  0001 C CNN
+F 1 "GND" V 4230 1472 50  0000 R CNN
+F 2 "" H 4225 1600 50  0001 C CNN
+F 3 "" H 4225 1600 50  0001 C CNN
+	1    4225 1600
 	0    1    1    0
 $EndComp
@@
 Text Label 7075 2100 0    50   ~ 0
 Q1E
+Text Label 7075 2500 0    50   ~ 0
+Q2C
+Text Label 6775 2300 0    50   ~ 0
+Q2B
+Text Label 5000 1950 1    50   ~ 0
+Q4B
+Text Label 4700 2150 0    50   ~ 0
+Q4C
+Text Label 4700 2350 0    50   ~ 0
+Q5B
+Text Label 4400 2150 0    50   ~ 0
+Q5C
+Text Label 6100 2700 1    50   ~ 0
+Q3B
+Wire Wire Line
+	5525 2700 5775 2700
+Wire Wire Line
+	5975 2700 6100 2700
+Text Label 6400 2500 0    50   ~ 0
+Q3C
+$Comp
+L 74xx:74HC14 U1
+U 7 1 5EC5A113
+P 4300 1100
+F 0 "U1" V 3933 1100 50  0000 C CNN
+F 1 "74HC14" V 4024 1100 50  0000 C CNN
+F 2 "" H 4300 1100 50  0001 C CNN
+F 3 "http://www.ti.com/lit/gpn/sn74HC14" H 4300 1100 50  0001 C CNN
+	7    4300 1100
+	0    1    1    0
+$EndComp
+Wire Wire Line
+	3800 1100 3800 1525
+Wire Wire Line
+	3800 1525 4225 1525
+Wire Wire Line
+	4225 1525 4225 1600
+Wire Wire Line
+	4225 1600 4300 1600
+Connection ~ 4225 1600
+Wire Wire Line
+	4400 1600 4800 1600
+Wire Wire Line
+	4800 1100 4800 1600
+Connection ~ 4400 1600
 $EndSCHEMATC
